Commit message: Add base_footprint as the URDF root (#9)
base_footprint sits on the ground directly under base_link (0.2032 m below), joined by a fixed joint. diff_drive_controller now uses it as base_frame_id, so odometry is odom -> base_footprint. The root has no inertia, which also removes robot_state_publisher's KDL root-inertia warning.

The spawn z argument now places base_footprint, so its default drops from 0.25 to 0.05 (same 5 cm settle) and the indoor example from 0.70 to 0.50. Docs and README updated to match.

File: src/aplc_description/urdf/aplc.urdf.xacro (robot description, xacro)
@@ -24,4 +24,12 @@
   <xacro:property name="wheel_y" value="${(overall_width - wheel_width) / 2}"/>
   <xacro:property name="wheel_z" value="${-height / 2}"/>
+  <!-- Root frame on the ground, directly under the chassis center (REP 105). Planar
+       navigation and the EKF track this frame; base_link sits above it. -->
+  <link name="base_footprint"/>
+  <joint name="base_footprint_joint" type="fixed">
+    <parent link="base_footprint"/>
+    <child link="base_link"/>
+    <origin xyz="0 0 ${height / 2 + wheel_radius}"/>
+  </joint>
   <!-- Main chassis -->
   <link name="base_link">
